Commit message: add multi robot.

File: description/urdf/pioneer3at-multi.urdf (robot description, URDF)
Before this commit: robot pioneer3at, 19 links, 18 joints
Links:
- removed link back_sonar
- removed link base_link
- removed link base_scan
- removed link front_sonar
- removed link left_cam_link
- removed link p3at_back_left_axle
- removed link p3at_back_left_hub
- removed link p3at_back_left_wheel
- removed link p3at_back_right_axle
- removed link p3at_back_right_hub
- removed link p3at_back_right_wheel
- removed link p3at_front_left_axle
- removed link p3at_front_left_hub
- removed link p3at_front_left_wheel
- removed link p3at_front_right_axle
- removed link p3at_front_right_hub
- removed link p3at_front_right_wheel
- removed link right_cam_link
- removed link top_plate
- added link $(arg ns)/back_sonar, mass 0.1; visual mesh filename=package://amr_robots_description/meshes/p3at_meshes/back_so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
- added link $(arg ns)/base_link, mass 21.5; collision mesh filename=package://amr_robots_description/meshes/p3at_meshes/chassis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; visual mesh filename=package://amr_robots_description/meshes/p3at_meshes/chassis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
- added link $(arg ns)/base_scan, mass 1e-5; collision box size=0.1 0.1 0.1; visual mesh filename=package://amr_robots_description/meshes/hokuyo/hokuyo.dae
- added link $(arg ns)/front_sonar, mass 0.1; visual mesh filename=package://amr_robots_description/meshes/p3at_meshes/front_s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
- added link $(arg ns)/p3at_back_left_axle, mass 0.1; collision mesh filename=package://amr_robots_description/meshes/p3at_meshes/axle.stl; visual mesh filename=package://amr_robots_description/meshes/p3at_meshes/axle.stl
- added link $(arg ns)/p3at_back_left_hub, mass 0.1; collision mesh filename=package://amr_robots_description/meshes/p3at_meshes/left_hu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; visual mesh filename=package://amr_robots_description/meshes/p3at_meshes/left_hu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
- added link $(arg ns)/p3at_back_left_wheel, mass 1.2; collision cylinder length=0.075 radius=0.111; visual mesh filename=package://amr_robots_description/meshes/p3at_meshes/wheel.s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
- added link $(arg ns)/p3at_back_right_axle, mass 0.1; collision mesh filename=package://amr_robots_description/meshes/p3at_meshes/axle.stl; visual mesh filename=package://amr_robots_description/meshes/p3at_meshes/axle.stl
- added link $(arg ns)/p3at_back_right_hub, mass 0.1; collision mesh filename=package://amr_robots_description/meshes/p3at_meshes/right_h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; visual mesh filename=package://amr_robots_description/meshes/p3at_meshes/right_h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
- added link $(arg ns)/p3at_back_right_wheel, mass 1.2; collision cylinder length=0.075 radius=0.111; visual mesh filename=package://amr_robots_description/meshes/p3at_meshes/wheel.s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
- added link $(arg ns)/p3at_front_left_axle, mass 0.1; visual mesh filename=package://amr_robots_description/meshes/p3at_meshes/axle.stl
- added link $(arg ns)/p3at_front_left_hub, mass 0.1; visual mesh filename=package://amr_robots_description/meshes/p3at_meshes/left_hu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
- added link $(arg ns)/p3at_front_left_wheel, mass 1.2; collision cylinder length=0.075 radius=0.111; visual mesh filename=package://amr_robots_description/meshes/p3at_meshes/wheel.s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
- added link $(arg ns)/p3at_front_right_axle, mass 0.1; visual mesh filename=package://amr_robots_description/meshes/p3at_meshes/axle.stl
- added link $(arg ns)/p3at_front_right_hub, mass 0.1; visual mesh filename=package://amr_robots_description/meshes/p3at_meshes/right_h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
- added link $(arg ns)/p3at_front_right_wheel, mass 1.2; collision cylinder length=0.075 radius=0.111; visual mesh filename=package://amr_robots_description/meshes/p3at_meshes/wheel.s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
- added link $(arg ns)/top_plate, mass 0.1; visual mesh filename=package://amr_robots_description/meshes/p3at_meshes/top.stl
Joints:
- removed joint base_back_joint
- removed joint base_front_joint
- removed joint base_front_left_axle_joint
- removed joint base_front_left_hub_joint
- removed joint base_front_right_axle_joint
- removed joint base_front_right_hub_joint
- removed joint base_leftcam_joint
- removed joint base_rightcam_joint
- removed joint base_top_joint
- removed joint hokuyo_joint
- removed joint p3at_back_left_axle_joint
- removed joint p3at_back_left_hub_joint
- removed joint p3at_back_left_wheel_joint
- removed joint p3at_back_right_axle_joint
- removed joint p3at_back_right_hub_joint
- removed joint p3at_back_right_wheel_joint
- removed joint p3at_front_left_wheel_joint
- removed joint p3at_front_right_wheel_joint
- added joint $(arg ns)/base_back_joint: type fixed, parent $(arg ns)/base_link, child $(arg ns)/back_sonar, origin xyz=-0.187 0 0.247 rpy=0 0 0
- added joint $(arg ns)/base_front_joint: type fixed, parent $(arg ns)/base_link, child $(arg ns)/front_sonar, origin xyz=0.193 0 0.25 rpy=0 0 0
- added joint $(arg ns)/base_front_left_axle_joint: type fixed, parent $(arg ns)/base_link, child $(arg ns)/p3at_front_left_axle, origin xyz=0.135 0.156 0.111 rpy=0 0 0
- added joint $(arg ns)/base_front_left_hub_joint: type fixed, parent $(arg ns)/p3at_front_left_axle, child $(arg ns)/p3at_front_left_hub, origin xyz=0 0.041 0 rpy=0 0 0
- added joint $(arg ns)/base_front_right_axle_joint: type fixed, parent $(arg ns)/base_link, child $(arg ns)/p3at_front_right_axle, origin xyz=0.135 -0.156 0.111 rpy=0 0 0
- added joint $(arg ns)/base_front_right_hub_joint: type fixed, parent $(arg ns)/p3at_front_right_axle, child $(arg ns)/p3at_front_right_hub, origin xyz=0 -0.041 0 rpy=0 0 0
- added joint $(arg ns)/base_top_joint: type fixed, parent $(arg ns)/base_link, child $(arg ns)/top_plate, origin xyz=0.003 0 0.274 rpy=0 0 0
- added joint $(arg ns)/hokuyo_joint: type fixed, parent $(arg ns)/base_link, child $(arg ns)/base_scan, origin xyz=0 0 0.33 rpy=0 0 0, axis 0 1 0
- added joint $(arg ns)/p3at_back_left_axle_joint: type fixed, parent $(arg ns)/base_link, child $(arg ns)/p3at_back_left_axle, origin xyz=-0.134 0.156 0.111 rpy=0 0 0
- added joint $(arg ns)/p3at_back_left_hub_joint: type fixed, parent $(arg ns)/p3at_back_left_axle, child $(arg ns)/p3at_back_left_hub, origin xyz=-0 0.041 0 rpy=0 0 0
- added joint $(arg ns)/p3at_back_left_wheel_joint: type continuous, parent $(arg ns)/p3at_back_left_hub, child $(arg ns)/p3at_back_left_wheel, origin xyz=0 0 0 rpy=0 0 0, axis 0 1 0, limit effort=100 velocity=100
- added joint $(arg ns)/p3at_back_right_axle_joint: type fixed, parent $(arg ns)/base_link, child $(arg ns)/p3at_back_right_axle, origin xyz=-0.134 -0.156 0.111 rpy=0 0 0
- added joint $(arg ns)/p3at_back_right_hub_joint: type fixed, parent $(arg ns)/p3at_back_right_axle, child $(arg ns)/p3at_back_right_hub, origin xyz=-0 -0.041 0 rpy=0 0 0
- added joint $(arg ns)/p3at_back_right_wheel_joint: type continuous, parent $(arg ns)/p3at_back_right_hub, child $(arg ns)/p3at_back_right_wheel, origin xyz=0 0 0 rpy=0 0 0, axis 0 1 0, limit effort=100 velocity=100
- added joint $(arg ns)/p3at_front_left_wheel_joint: type continuous, parent $(arg ns)/p3at_front_left_hub, child $(arg ns)/p3at_front_left_wheel, origin xyz=0 0 0 rpy=0 0 0, axis 0 1 0, limit effort=100 velocity=100
- added joint $(arg ns)/p3at_front_right_wheel_joint: type continuous, parent $(arg ns)/p3at_front_right_hub, child $(arg ns)/p3at_front_right_wheel, origin xyz=0 0 0 rpy=0 0 0, axis 0 1 0, limit effort=100 velocity=100

Commit message: add more training sectors.

File: description/urdf/pioneer3at-multi.urdf (robot description, URDF)
Before this commit: robot pioneer3at, 17 links, 16 joints
Joints:
- joint $(arg ns)/hokuyo_joint: axis 0 1 0 -> (none); origin xyz=0 0 0.33 rpy=0 0 0 -> xyz=0 0 0.5 rpy=0 0 0

File: description/urdf/pioneer3at.urdf (robot description, URDF)
Before this commit: robot pioneer3at, 19 links, 18 joints
Links:
- added link velodyne, mass 0.01; visual mesh filename=package://velodyne_description/meshes/VLP16_base_1.dae; visual mesh filename=package://velodyne_description/meshes/VLP16_base_2.dae
Joints:
- added joint base_velodyne_joint: type fixed, parent base_link, child velodyne, origin xyz=0 0 0.5 rpy=0 0 0
