Commit message: add hokuyo,velodyne,camera. add a sample road.

File: description/urdf/pioneer3at.urdf (robot description, URDF)
Before this commit: robot pioneer3at, 16 links, 15 joints
Links:
- added link cam_link, mass 0.1; visual mesh filename=package://amr_robots_description/meshes/xtion/asus_xtion_pr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
Joints:
- added joint base_cam_joint: type fixed, parent base_link, child cam_link, origin xyz=0.2 0 0.35 rpy=0 0 0

Commit message: add some tools for keyboard and use semantic seg.

File: description/urdf/pioneer3at.urdf (robot description, URDF)
Before this commit: robot pioneer3at, 17 links, 16 joints
Joints:
- joint base_cam_joint: origin xyz=0.2 0 0.35 rpy=0 0 0 -> xyz=0.2 0 1.2 rpy=0 0.2 0

Commit message: [nav]add a simulation using movebase provided by ros.

File: description/urdf/pioneer3at.urdf (robot description, URDF)
Before this commit: robot pioneer3at, 17 links, 16 joints
Links:
- added link base_scan, mass 1e-5; collision box size=0.1 0.1 0.1; visual mesh filename=package://amr_robots_description/meshes/hokuyo/hokuyo.dae
Joints:
- added joint hokuyo_joint: type fixed, parent base_link, child base_scan, origin xyz=0 0 0.33 rpy=0 0 0, axis 0 1 0

Commit message: add depth cam. modify some param.

File: description/urdf/pioneer3at.urdf (robot description, URDF)
Before this commit: robot pioneer3at, 18 links, 17 joints
Links:
- removed link cam_link
- added link left_cam_link, mass 0.1
- added link right_cam_link, mass 0.1
Joints:
- removed joint base_cam_joint
- added joint base_leftcam_joint: type fixed, parent base_link, child left_cam_link, origin xyz=0.2 0.1 1 rpy=0 0 0
- added joint base_rightcam_joint: type fixed, parent base_link, child right_cam_link, origin xyz=0.2 -0.1 1 rpy=0 0 0

Commit message: modify for elevation map.

File: description/urdf/pioneer3at.urdf (robot description, URDF)
Before this commit: robot pioneer3at, 20 links, 19 joints
Links:
- added link kinect_link, mass 0.0001; visual mesh filename=package://amr_robots_description/meshes/xtion/asus_xtion_pr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
Joints:
- added joint base_kinect_joint: type fixed, parent base_link, child kinect_link, origin xyz=0.2 0.0 0.5 rpy=0 0 0
